File: Hardware/Qwiic_PIR.sch (EAGLE design)
At the start: 29 parts, among them J2 QWIIC, J3 QWIIC, J7 ISP, U1 EKMC4607112k, U4 ATTINY84-ARDUINO

Commit message: post checklist changes
Parts:
- removed JP1, JP4: JUMPER-SMT_2_NC_TRACE_SILK, SparkFun-Jumpers:JUMPER-SMT_2_NC_TRACE_SILK
- removed JP3: JUMPER-SMT_3_2-NC_TRACE_SILK, SparkFun-Jumpers:JUMPER-SMT_3_2-NC_TRACE_SILK
- added ADR, PWR: JUMPER-SMT_2_NC_TRACE_SILK, SparkFun-Jumpers:JUMPER-SMT_2_NC_TRACE_SILK
- added D2: 24V, SparkFun-DiscreteSemi:DIODE_TVS
- added I2C: JUMPER-SMT_3_2-NC_TRACE_SILK, SparkFun-Jumpers:JUMPER-SMT_3_2-NC_TRACE_SILK
- added LOGO2: QWIIC_LOGO_5MM, SparkFun-Aesthetics:QWIIC_LOGO_5MM
Connections:
- net 3.3V: now also D2.C, I2C.2, PWR.2; no longer JP3.2, JP4.2
- net ADR0: now also ADR.2; no longer JP1.2
- net GND: now also ADR.1, D2.A; no longer JP1.1
- net SCL_PU1: now also I2C.1; no longer JP3.1
- net SDA_PU1: now also I2C.3; no longer JP3.3
- net STAT: now also PWR.1; no longer JP4.1
Other:
- note added: "Cut the ADR jumper to change the address of the PIR from 0x12(Default) to 0x13"
- note added: "Cut the PWR jumper to disbale the PWR LED"
- note added: "This PIR sensor is different between 170 uA (IC-15368) and 1uA (IC-15370) versions"
- note added: "VIN: 2.3-4.0V"
- note removed: "Address Jumpers"
- note removed: "Cut the ADR jumper to change the address of the PIR from 0x12 to 0x13"
- moved on the sheet: C2, D1, J7, R1, R2, R3, R4, U4
